File: Project Fauxbow/Project Fauxbow.kicad_pcb (KiCad board)
At the start: 2 copper layers, 126.4 x 104.8 mm, 65 parts, among them J1 Host, J2 USB 1, J3 USB 2, J4 USB 3, K1 Kailh Hotswap Socket, K10 Kailh Hotswap Socket, K11 Kailh Hotswap Socket, K12 Kailh Hotswap Socket, K13 Kailh Hotswap Socket, K14 Kailh Hotswap Socket, K15 Kailh Hotswap Socket, K16 Kailh Hotswap Socket, K17 Kailh Hotswap Socket, K18 Kailh Hotswap Socket, K19 Kailh Hotswap Socket, K2 Kailh Hotswap Socket, K20 Kailh Hotswap Socket, K3 Kailh Hotswap Socket, K4 Kailh Hotswap Socket, K5 Kailh Hotswap Socket, K6 Kailh Hotswap Socket, K7 Kailh Hotswap Socket, K8 Kailh Hotswap Socket, K9 Kailh Hotswap Socket, SW1 SW_Push, U1 ATmega32U4-A, U2 AP1117-33, U3 FE1.1, Y1 16MHz, Y2 12MHz

Commit message: INITIAL COMMIT REV 1
Parts:
- removed C1, C2: 22pF, Capacitor_SMD:C_1206_3216Metric_Pad1.33x1.80mm_HandSolder
- removed C3, C4: 10u, Capacitor_SMD:C_0805_2012Metric
- removed J1: Host, Connector_USB:USB_C_Receptacle_Palconn_UTC16-G
- removed J2: USB 1, Connector_USB:USB_A_Stewart_SS-52100-001_Horizontal
- removed J3: USB 2, Connector_USB:USB_A_Stewart_SS-52100-001_Horizontal
- removed J4: USB 3, Connector_USB:USB_A_Stewart_SS-52100-001_Horizontal
- removed R1: 10k, Resistor_SMD:R_1206_3216Metric_Pad1.30x1.75mm_HandSolder
- removed R3, R4: 5.1k, Resistor_SMD:R_0805_2012Metric
- removed R5: 2.7k, Resistor_SMD:R_0805_2012Metric
- removed U1: ATmega32U4-A, Package_QFP:TQFP-44_10x10mm_P0.8mm
- removed U2: AP1117-33, Package_TO_SOT_SMD:SOT-223-3_TabPin2
- removed U3: FE1.1, Package_QFP:LQFP-48_7x7mm_P0.5mm
- removed Y1: 16MHz, Oscillator:Oscillator_SMD_Abracon_ASE-4Pin_3.2x2.5mm_HandSoldering
- removed Y2: 12MHz, Crystal:Crystal_SMD_3225-4Pin_3.2x2.5mm
- added U4: Elite-C, keebs:Elite-C-castellated-29pin-holes, F.Cu at (163.3, 75.5)
- moved SW1 107.5 mm to (149.5, 95.4), turned to 90 degrees
- moved H1 48.6 mm to (114.5, 90.0)
Routing:
- net VBUS: track 675.7 -> 445.5 mm, vias 25 -> 20
- net key_15: track 78.6 -> 219.5 mm, vias 1 -> 4
- net 4D+: track 119.9 -> 0.00 mm, vias 4 -> 0
- net 4D-: track 115.0 -> 0.00 mm, vias 2 -> 0
- net key_10: track 107.7 -> 198.6 mm, vias 1 -> 5
- net GND: track 769.8 -> 682.3 mm, vias 12 -> 0
- net Net-(D31-Pad1): track 81.6 -> 167.9 mm, vias 0 -> 2
- net key_16: track 132.4 -> 61.0 mm, vias 4 -> 5
- net key_20: track 165.6 -> 95.7 mm, vias 1 -> 6
- net reset: track 100.0 -> 30.5 mm, vias 5 -> 0
- net key_17: track 133.9 -> 72.8 mm, vias 5 -> 6
- net key_19: track 55.1 -> 0.00 mm, vias 1 -> 0
- net key_13: track 51.8 -> 0.83 mm, vias 7 -> 0
- net key_11: track 28.6 -> 78.6 mm, vias 1 -> 0
- net +3V3: track 49.9 -> 0.00 mm, vias 3 -> 0
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- removed copper zone on B.Cu, net (none)
- removed copper zone on F.Cu, net (none)
- removed copper zone on B.Cu, net GND
- removed copper zone on F.Cu, net GND
